File: Schematics/Cluster.sch (KiCad schematic (older format))
At the start: 34 parts, among them J1 FairingConnector, J10 PowerReg, J11 Conn_01x02, J12 Conn_01x03, J2 Serial, J3 i2c, J4 Programming, J5 GPIO, J6 Conn_01x07, J7 Conn_01x40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

Commit message: Added missing time IC and turn signal inputs to schematic
Parts:
- added BT1: Battery_Cell, symbol Device:Battery_Cell
- added C11, C12: 20pF, Capacitors_SMD:C_0805, symbol Device:C_Small
- added C13, C14, C15: 10uF, Capacitors_SMD:C_0805, symbol Device:C_Small
- added C16: 0.1uF, Capacitors_SMD:C_0805, symbol Device:C_Small
- added D2, D3: D_ALT, symbol Device:D_ALT
- added J13: ClkOUT, Pin_Headers:Pin_Header_Straight_1x01_Pitch2.54mm, symbol Connector_Generic:Conn_01x01
- added J14: Conn_01x02, symbol Connector_Generic:Conn_01x02
- added R7: 1k, Resistors_SMD:R_0805, symbol Device:R_Small
- added U4: AiP8563, symbol Cluster:AiP8563
- added U5: badge-rescue_HX4056, symbol badge-cache:badge-rescue_HX4056
- added Y2: 32.768kHz, symbol Device:Crystal_Small
- U1: symbol LIS3DHTR:LIS3DHTR -> Cluster-rescue:LIS3DHTR-LIS3DHTR
Connections:
- net SCL: now also U4.6 (SCL)
- net SDA: now also U4.5 (SDA)
- net VCC: now also C13.2, D3.2 (A), U5.4 (Vin)
- net VSS: now also BT1.2 (-), C11.2, C12.2, C13.1, C15.1, R7.1, U4.4 (VSS), U5.3 (GND), U5.9 (GND)
- net LeftIN: now reaches U3.40 (PC9)
- net LeftIN: now also J14.2 (Pin_2)
- net RightIN: now reaches U3.41 (PA8)
- net RightIN: now also J14.1 (Pin_1)
- new net: C11.1, U4.1 (OSCI), Y2.1
- new net: C12.1, U4.2 (OSCO), Y2.2
- new net: J13.1 (Pin_1), U4.7 (CLKOUT)
- new net: C14.2, C16.2, D2.1 (K), D3.1 (K), U4.8 (VDD)
- new net: BT1.1 (+), C15.2, D2.2 (A), U5.5 (BAT)
- new net: R7.2, U5.2 (ISET)
- no-connect marks 19 -> 20
Other:
- moved on the sheet: C1, C4, C5, D1, J10, L1, R1, R2, R3, R4, U2
