File: Schematics/Cluster/Cluster.kicad_pcb (KiCad board)
At the start: 2 copper layers, 100 x 74 mm, 65 parts, among them J1 FairingConnector, J10 PowerReg, J11 Conn_01x02, J12 Conn_01x03, J13 ClkOUT, J14 Conn_01x02, J2 Serial, J3 i2c, J4 Programming, J5 GPIO, J6 Conn_01x07, J7 Conn_01x40, J8 Conn_01x40, J9 Conn_01x03, U1 LIS3DHTR, U2 LM2596S-ADJ, U3 STM32F411RETx, U4 AiP8563, U5 badge-rescue_HX4056, Y1 8MHz, Y2 32.768kHz

Commit message: Ordered V2
Parts:
- removed the C2 at (177.0, 123.5)
- removed the C3 at (173.0, 123.5)
- removed the C6 at (149.0, 102.5)
- removed the J8 at (203.5, 101.1)
- removed the R2 at (161.0, 99.5)
- removed the R6 at (154.9, 111.5)
- added C11: 100nF, Capacitor_SMD:C_0805_2012Metric, F.Cu at (172.5, 123.6)
- added C12: 100nF, Capacitor_SMD:C_0805_2012Metric, F.Cu at (179.1, 97.8)
- added C14: 100nF, Capacitor_SMD:C_0805_2012Metric, F.Cu at (163.2, 121.4)
- added C17: 4.7uF, Capacitor_SMD:C_0805_2012Metric, F.Cu at (172.3, 103.3)
- added C21: 20pF, Capacitors_SMD:C_0805, F.Cu at (149.0, 102.5)
- added C23: 1.5pF, Capacitor_SMD:C_0805_2012Metric, F.Cu at (160.8, 103.2)
- added C24: 1.5pF, Capacitor_SMD:C_0805_2012Metric, F.Cu at (161.0, 101.2)
- added C4: 100nF, Capacitor_SMD:C_0805_2012Metric, F.Cu at (160.9, 105.2)
- added C5: 100nF, Capacitor_SMD:C_0805_2012Metric, F.Cu at (154.9, 119.2)
- added C7: 100nF, Capacitor_SMD:C_0805_2012Metric, F.Cu at (163.5, 104.3)
- added C8: 1uF, Capacitor_SMD:C_0805_2012Metric, F.Cu at (154.9, 117.2)
- added C9: 100nF, Capacitor_SMD:C_0805_2012Metric, F.Cu at (172.3, 106.3)
- added D4: Pwr Ind, LED_SMD:LED_0603_1608Metric, F.Cu at (192.0, 85.5)
- added J15: Conn_01x02, TerminalBlock_RND:TerminalBlock_RND_205-00012_1x02_P5.00mm_Horizontal, F.Cu at (153.7, 71.8)
- added J7: Conn_01x40, Cluster:XF2M-4015, F.Cu at (203.5, 101.1)
- added L2: L_Small, Inductor_SMD:L_0603_1608Metric, F.Cu at (154.8, 115.4)
- added R7: 330, Resistor_SMD:R_0603_1608Metric, F.Cu at (192.0, 89.1)
- added Y3: 32.768kHz, Crystal:Crystal_SMD_2012-2Pin_2.0x1.2mm, F.Cu at (157.8, 102.1)
- C10: value 100nF -> 10uF; footprint Capacitors_SMD:C_0805 -> Capacitor_SMD:C_0805_2012Metric
- J1: footprint TerminalBlock_RND:TerminalBlock_RND_205-00022_Pitch5.00mm -> TerminalBlock_RND:TerminalBlock_RND_205-00021_1x11_P5.00mm_Horizontal
- J4: footprint Pin_Headers:Pin_Header_Straight_1x07_Pitch2.54mm -> Connector_PinHeader_2.54mm:PinHeader_1x08_P2.54mm_Vertical
- J5: footprint Pin_Headers:Pin_Header_Straight_1x06_Pitch2.54mm -> Connector_PinHeader_2.54mm:PinHeader_1x06_P2.54mm_Vertical
- J6: value Conn_01x07 -> Conn_01x06; footprint Pin_Headers:Pin_Header_Straight_1x07_Pitch2.54mm -> Connector_PinHeader_2.54mm:PinHeader_1x06_P2.54mm_Vertical
- J9: renamed from J7; moved to B.Cu
- R5: value 100k -> 2k
- moved J9 40.5 mm to (197.9, 78.0)
- moved J10 35.6 mm to (192.9, 115.6), turned to 180 degrees
- moved C10 33.2 mm to (179.2, 94.8)
- moved J12 12.5 mm to (155.8, 88.0), turned to 270 degrees
- moved R5 12.1 mm to (163.2, 92.2)
- moved C19 7.62 mm to (159.7, 92.2)
- moved R4 7.62 mm to (166.7, 92.2)
- moved U2 4.93 mm to (160.8, 81.8), turned to 0 degrees
- moved J1 4.83 mm to (199.3, 130.9)
- moved BT1 3.92 mm to (222.8, 131.8)
- moved J6 2.73 mm to (151.5, 126.1)
- moved J5 1.12 mm to (145.6, 122.2)
- moved C25 0.81 mm to (154.9, 113.7)
- moved J4 0.14 mm to (145.6, 88.1)
- renumbered C14 to C13, C4 to C18, C5 to C19, C11 to C2, C17 to C20, C7 to C22, C8 to C25, C9 to C26, C18 to C27, C19 to C28, C20 to C29, C12 to C3, C21 to C30, C13 to C6, D4 to D5, D5 to D6, D6 to D7, D7 to D8, D8 to D9, J9 to J10, J10 to J12, J12 to J13, J13 to J14, J14 to J8, R8 to R1, R3 to R2, R7 to R3, R1 to R4, R4 to R6, U4 to U3, U5 to U4, U3 to U5, Y2 to Y1, Y1 to Y2
Connections:
- C10 pad 2: Net-(C10-Pad2) -> VSS
- C19 pad 1: Net-(C5-Pad1) -> Net-(C19-Pad1)
- J1 pad 1: +12V -> VCC
- J1 pad 10: Oil -> Fuel
- J1 pad 11: Fuel -> Neutral
- J1 pad 2: VCC -> VSS
- J1 pad 3: VSS -> HighBeam
- J1 pad 4: HighBeam -> RightTurn
- J1 pad 5: RightTurn -> LeftTurn
- J1 pad 6: LeftTurn -> OverDrive
- J1 pad 7: OverDrive -> LowFuel
- J1 pad 8: LowFuel -> Temp
- J1 pad 9: Temp -> Oil
- J10 pad 1: Net-(J7-Pad40) -> VCC
- J10 pad 2: Net-(J7-Pad39) -> VSS
- J10 pad 3: Net-(J7-Pad38) -> VCC
- J6 pad 1: +12V -> VCC
- J6 pad 2: VCC -> VSS
- J6 pad 3: VSS -> LightsOutAuxTwo
- J6 pad 4: LightsOutAuxTwo -> LightsOutAux
- J6 pad 5: LightsOutAux -> LightsOutBack
- J6 pad 6: LightsOutBack -> LightsOutFront
- J9 pad 38: Net-(J7-Pad38) -> VCC
- J9 pad 39: Net-(J7-Pad39) -> VSS
- J9 pad 40: Net-(J7-Pad40) -> VCC
- R4 pad 1: Net-(C5-Pad1) -> Net-(C19-Pad1)
- R5 pad 1: Net-(R5-Pad1) -> VSS
- R5 pad 2: VSS -> Net-(C19-Pad1)
- U2 pad 4: Net-(C5-Pad1) -> Net-(C19-Pad1)
- U5 pad 13: Net-(C10-Pad2) -> VDDA
- U5 pad 60: Net-(R5-Pad1) -> Boot0
Routing:
- net +12V: track 224.6 -> 15.3 mm, vias 1 -> 0
- net VCC: track 335.3 -> 389.1 mm, vias 11 -> 12
- net MISO: track 46.6 -> 10.5 mm, vias 1 -> 0
- net Net-(BT1-Pad1): track 116.1 -> 80.1 mm
- net MOSI: track 47.1 -> 11.4 mm, vias 1 -> 0
- net Boot0: track 0.00 -> 32.1 mm, vias 0 -> 2
- net Net-(C19-Pad1): track 0.00 -> 23.6 mm
- net VSS: track 116.8 -> 94.1 mm
- net GPIO6: track 22.5 -> 0.00 mm
- net Net-(J7-Pad38): track 21.3 -> 0.00 mm
- net Net-(J7-Pad39): track 20.9 -> 0.00 mm
- net Net-(J7-Pad40): track 20.6 -> 0.00 mm
- net SCK: track 42.8 -> 63.5 mm
- net Net-(J9-Pad37): track 15.2 -> 0.00 mm
- net Net-(C24-Pad1): track 0.00 -> 14.3 mm
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Other:
- board text added: "V2"
- board text removed: "GPIO5"
- board text removed: "GPIO6"
- board text removed: "V1"

Commit message: Why are there still ratsnest wires?
Connections:
- J4 pad 3: JRST -> Net-(J4-Pad3)
- J4 pad 4: SWO -> Net-(J4-Pad4)
- U5 pad 10: MISO -> Net-(U5-Pad10)
- U5 pad 11: MOSI -> Net-(U5-Pad11)
- U5 pad 29: SCK -> Net-(U5-Pad29)
- U5 pad 55: SWO -> SCK
- U5 pad 56: JRST -> MOSI
- U5 pad 57: Net-(U5-Pad57) -> MISO
Routing:
- net MISO: track 10.5 -> 53.7 mm, vias 0 -> 2
- net MOSI: track 11.4 -> 53.0 mm, vias 0 -> 3
- net GPIO6: track 0.00 -> 40.0 mm, vias 0 -> 1
- net JRST: track 28.5 -> 0.00 mm, vias 1 -> 0
- net SWO: track 28.5 -> 0.00 mm, vias 1 -> 0
- net Net-(J7-Pad7): track 0.00 -> 13.4 mm
- net VSS: track 94.1 -> 105.2 mm, vias 22 -> 25
- net VCC: track 389.1 -> 395.9 mm, vias 12 -> 14
- net SCK: track 63.5 -> 63.0 mm
